File: IOB_V3.kicad_sch (KiCad schematic)
At the start: 8 parts, among them J1 Conn_01x02, J2 Conn_01x03, U1 REF3033

Commit message: Ready for first review
Parts:
- added G1: SpaceTeam_LOGO, TXV_Library_Footprints:ST_Logo_new, symbol TXV_Library_Symbols:SpaceTeam_LOGO
- J18, J20: value (none) -> Conn_01x10; footprint (none) -> Connector_IDC:IDC-Header_2x05_P2.54mm_Vertical
Changed lines of the file:
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@@
   (symbol (lib_id "power:+3.3V") (at 87.63 165.862 0) (unit 1)
     (in_bom yes) (on_board yes)
-    (property "Reference" "#PWR?" (id 0) (at 87.63 169.672 0)
+    (property "Reference" "#PWR0149" (id 0) (at 87.63 169.672 0)
       (effects (font (size 1.27 1.27)) hide)
     )
@@
     (in_bom yes) (on_board yes)
     (property "Reference" "J20" (id 0) (at 115.57 176.276 0))
-    (property "Value" "" (id 1) (at 112.268 179.578 0))
-    (property "Footprint" "" (id 2) (at 120.142 178.054 0)
+    (property "Value" "Conn_01x10" (id 1) (at 112.268 179.578 0))
+    (property "Footprint" "Connector_IDC:IDC-Header_2x05_P2.54mm_Vertical" (id 2) (at 120.142 178.054 0)
       (effects (font (size 1.27 1.27)) hide)
     )
@@
     (in_bom yes) (on_board yes)
     (property "Reference" "J18" (id 0) (at 72.644 176.784 0))
-    (property "Value" "" (id 1) (at 67.056 180.594 0))
-    (property "Footprint" "" (id 2) (at 76.454 177.292 0)
+    (property "Value" "Conn_01x10" (id 1) (at 67.056 180.594 0))
+    (property "Footprint" "Connector_IDC:IDC-Header_2x05_P2.54mm_Vertical" (id 2) (at 76.454 177.292 0)
       (effects (font (size 1.27 1.27)) hide)
     )
@@
     (pin "1")
   )
+  (symbol (lib_id "TXV_Library_Symbols:SpaceTeam_LOGO") (at 62.484 85.471 0) (unit 1)
+    (in_bom yes) (on_board yes) (fields_autoplaced)
+    (property "Reference" "G1" (id 0) (at 62.484 90.7034 0)
+      (effects (font (size 1.524 1.524)) hide)
+    )
+    (property "Value" "SpaceTeam_LOGO" (id 1) (at 62.484 80.2386 0)
+      (effects (font (size 1.524 1.524)) hide)
+    )
+    (property "Footprint" "TXV_Library_Footprints:ST_Logo_new" (id 2) (at 62.484 85.471 0)
+      (effects (font (size 1.27 1.27)) hide)
+    )
+    (property "Datasheet" "" (id 3) (at 62.484 85.471 0)
+      (effects (font (size 1.27 1.27)) hide)
+    )
+  )
   (symbol (lib_id "power:GNDA") (at 236.982 86.995 0) (unit 1)
     (in_bom yes) (on_board yes)
@@
   (symbol (lib_id "power:+3.3V") (at 131.318 166.624 0) (unit 1)
     (in_bom yes) (on_board yes)
-    (property "Reference" "#PWR?" (id 0) (at 131.318 170.434 0)
+    (property "Reference" "#PWR0148" (id 0) (at 131.318 170.434 0)
       (effects (font (size 1.27 1.27)) hide)
     )
@@
     )
     (pin "1")
-  )
-  (symbol (lib_id "TXV_Library_Symbols:SpaceTeam_LOGO") (at 68.326 94.615 0) (unit 1)
-    (in_bom yes) (on_board yes) (fields_autoplaced)
-    (property "Reference" "#G1" (id 0) (at 68.326 99.8474 0)
-      (effects (font (size 1.524 1.524)) hide)
-    )
-    (property "Value" "SpaceTeam_LOGO" (id 1) (at 68.326 89.3826 0)
-      (effects (font (size 1.524 1.524)) hide)
-    )
-    (property "Footprint" "" (id 2) (at 68.326 94.615 0)
-      (effects (font (size 1.27 1.27)) hide)
-    )
-    (property "Datasheet" "" (id 3) (at 68.326 94.615 0)
-      (effects (font (size 1.27 1.27)) hide)
-    )
   )
   (symbol (lib_id "Device:C") (at 81.661 147.828 0) (unit 1)
@@
       (reference "#FLG0101") (unit 1) (value "PWR_FLAG") (footprint "")
     )
-    (path "/ac4c4951-e08c-483f-aab9-5cd115cbd241"
-      (reference "#G1") (unit 1) (value "SpaceTeam_LOGO") (footprint "TXV_Library_Footprints:ST_Logo_new")
-    )
     (path "/00c5ccef-eb29-45b1-8f65-055873a11b7e"
       (reference "#PWR01") (unit 1) (value "GND") (footprint "")
@@
       (reference "#PWR0147") (unit 1) (value "GNDA") (footprint "")
     )
+    (path "/9dbe0d25-4225-40ae-a49f-c30c39c46cfe"
+      (reference "#PWR0148") (unit 1) (value "+3.3V") (footprint "")
+    )
+    (path "/0a9d8e41-616b-478b-a794-2d1c96fc98c8"
+      (reference "#PWR0149") (unit 1) (value "+3.3V") (footprint "")
+    )
     (path "/534d7b1f-d272-47da-b7a1-47aab2c48175/49ac7742-282c-4f80-a888-ce3f270663b8"
       (reference "#PWR0155") (unit 1) (value "GNDD") (footprint "")
@@
       (reference "#PWR0161") (unit 1) (value "+3.3V") (footprint "")
     )
-    (path "/0a9d8e41-616b-478b-a794-2d1c96fc98c8"
-      (reference "#PWR?") (unit 1) (value "+3.3V") (footprint "")
-    )
-    (path "/9dbe0d25-4225-40ae-a49f-c30c39c46cfe"
-      (reference "#PWR?") (unit 1) (value "+3.3V") (footprint "")
-    )
     (path "/b53ac17e-5879-4554-b7b4-15c13cd6c313"
       (reference "C1") (unit 1) (value "100n") (footprint "Capacitor_SMD:C_0402_1005Metric")
@@
       (reference "F25") (unit 1) (value "Polyfuse") (footprint "TXV_Library_Footprints:0805L110SL PPTC Polyfuse Littelfuse")
     )
+    (path "/9c27bafe-dc9a-4fc8-9304-3713da742e75"
+      (reference "G1") (unit 1) (value "SpaceTeam_LOGO") (footprint "TXV_Library_Footprints:ST_Logo_new")
+    )
     (path "/3bbae5d4-6082-49cc-a334-20e15dfcb8e0"
