File: 24V_to_5V-12V_SMPS.kicad_sch (KiCad schematic)
At the start: 10 parts, among them U14 TS30041

Commit message: WIP
Changed lines of the file:
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@@
   (junction (at 140.97 129.54) (diameter 0) (color 0 0 0 0)
-  )
-  (junction (at 121.92 96.52) (diameter 0) (color 0 0 0 0)
   )
   (junction (at 193.04 124.46) (diameter 0) (color 0 0 0 0)
   )
   (junction (at 165.1 104.14) (diameter 0) (color 0 0 0 0)
+  )
+  (junction (at 121.92 96.52) (diameter 0) (color 0 0 0 0)
   )
   (junction (at 185.42 96.52) (diameter 0) (color 0 0 0 0)
@@
     (stroke (width 0) (type default) (color 0 0 0 0))
   )
+  (wire (pts (xy 121.92 96.52) (xy 124.46 96.52))
+    (stroke (width 0) (type default) (color 0 0 0 0))
+  )
   (wire (pts (xy 193.04 96.52) (xy 193.04 110.49))
     (stroke (width 0) (type default) (color 0 0 0 0))
@@
     (stroke (width 0) (type default) (color 0 0 0 0))
   )
-  (wire (pts (xy 124.46 96.52) (xy 121.92 96.52))
-    (stroke (width 0) (type default) (color 0 0 0 0))
-  )

Commit message: Schematic nearly complete
Changed lines of the file:
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@@
     (effects (font (size 1.27 1.27)) (justify left))
+  )
+  (symbol (lib_id "power:PWR_FLAG") (at 121.92 96.52 0) (unit 1)
+    (in_bom yes) (on_board yes) (fields_autoplaced)
+    (property "Reference" "#FLG0101" (id 0) (at 121.92 94.615 0)
+      (effects (font (size 1.27 1.27)) hide)
+    )
+    (property "Value" "PWR_FLAG" (id 1) (at 121.92 91.44 0)
+      (effects (font (size 1.27 1.27)) hide)
+    )
+    (property "Footprint" "" (id 2) (at 121.92 96.52 0)
+      (effects (font (size 1.27 1.27)) hide)
+    )
+    (property "Datasheet" "~" (id 3) (at 121.92 96.52 0)
+      (effects (font (size 1.27 1.27)) hide)
+    )
+    (pin "1")
   )
   (symbol (lib_id "power:PWR_FLAG") (at 193.04 96.52 0) (unit 1)

Commit message: Routing begin
Parts:
- F25: footprint Fuse:Fuse_Littelfuse-LVR125 -> TXV_Library_Footprints:0805L110SL PPTC Polyfuse Littelfuse
Changed lines of the file:
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@@
       (effects (font (size 1.27 1.27)) (justify left))
     )
-    (property "Footprint" "Fuse:Fuse_Littelfuse-LVR125" (id 2) (at 102.87 95.25 0)
+    (property "Footprint" "TXV_Library_Footprints:0805L110SL PPTC Polyfuse Littelfuse" (id 2) (at 102.87 95.25 0)
       (effects (font (size 1.27 1.27)) (justify left) hide)
     )

Commit message: Fixed Lib Mess
Parts:
- U14: footprint Package_DFN_QFN:QFN-16-1EP_3x3mm_P0.5mm_EP1.9x1.9mm_ThermalVias -> Package_DFN_QFN:QFN-16-1EP_3x3mm_P0.5mm_EP1.75x1.75mm_ThermalVias; symbol IOB-rescue:TS30041-TXV_Library_Symbols -> TXV_Library_Symbols:TS30041
Changed lines of the file:
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@@
     (pin "2")
   )
-  (symbol (lib_id "IOB-rescue:TS30041-TXV_Library_Symbols") (at 139.7 107.95 0) (unit 1)
+  (symbol (lib_id "TXV_Library_Symbols:TS30041") (at 139.7 107.95 0) (unit 1)
     (in_bom yes) (on_board yes)
     (property "Reference" "U14" (id 0) (at 139.7 89.789 0))
     (property "Value" "TS30041" (id 1) (at 139.7 92.1004 0))
-    (property "Footprint" "Package_DFN_QFN:QFN-16-1EP_3x3mm_P0.5mm_EP1.9x1.9mm_ThermalVias" (id 2) (at 138.43 137.16 0)
+    (property "Footprint" "Package_DFN_QFN:QFN-16-1EP_3x3mm_P0.5mm_EP1.75x1.75mm_ThermalVias" (id 2) (at 138.43 137.16 0)
       (effects (font (size 1.524 1.524)) hide)
     )
